File: kick-drum.kicad_pcb (KiCad board)
At the start: 2 copper layers, 63 x 128.5 mm, 69 parts, among them J1 Conn_02x05_Odd_Even, J2 GATE, J3 ACCENT CV, J4 PITCH CV, J5 OUTPUT, Q1 BCM857DS,135, Q2 BC547C, Q3 BCM847DS,135, U1 TL074

Commit message: v0 ready
Parts:
- moved H13 91.0 mm to (113.7, 137.5)
- moved H14 91.0 mm to (113.7, 143.3)
- moved H15 91.0 mm to (113.7, 149.1)
- moved H9 91.0 mm to (109.6, 168.4)
- moved H1 91.0 mm to (91.6, 107.1)
- moved H10 91.0 mm to (109.6, 182.1)
- moved H11 91.0 mm to (109.6, 195.8)
- moved H12 91.0 mm to (109.6, 212.4)
- moved H2 91.0 mm to (111.6, 107.1)
- moved H3 91.0 mm to (111.6, 229.6)
- moved H4 91.0 mm to (91.6, 229.6)
- moved H5 91.0 mm to (95.6, 122.4)
- moved H6 91.0 mm to (95.6, 148.4)
- moved H7 91.0 mm to (95.6, 174.4)
- moved H8 91.0 mm to (95.6, 200.4)
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Connections:
- RV2 pad 1: Net-(Q3B-E2) -> Net-(R13-Pad1)
- RV2 pad 3: Net-(R13-Pad1) -> Net-(Q3B-E2)
- RV7 pad 1: Net-(D6-K) -> Net-(D6-A)
- RV7 pad 3: Net-(D6-A) -> Net-(D6-K)
Routing:
- net Net-(D6-K): track 32.2 -> 14.9 mm
- net Net-(Q3B-E2): track 17.2 -> 12.1 mm
- net Net-(R13-Pad1): track 6.52 -> 9.92 mm
- net /GATE: track 4.00 -> 2.55 mm
- net Net-(U1C--): track 39.7 -> 38.5 mm
- net +12V: track 78.5 -> 77.8 mm
- net Net-(R18-Pad2): track 35.6 -> 34.9 mm
- net GND: track 125.5 -> 125.0 mm
- net Net-(Q1B-E2): track 8.45 -> 7.93 mm
Other:
- board size 63 x 128.5 mm -> 30 x 232.4 mm
- board text added: "kick"
- board text added: "thismatters/kick-drum/v0"
