File: kick-drum.kicad_sch (KiCad schematic)
At the start: 73 parts, among them J1 Conn_02x05_Odd_Even, J2 GATE, J3 ACCENT CV, J4 PITCH CV, J5 OUTPUT, Q1 BCM857DS,135, Q2 BC547C, Q3 BCM847DS,135, U1 TL074

Commit message: v1 ready
Parts:
- removed Q2: BC547C, Package_TO_SOT_SMD:SOT-23-3, symbol Device:Q_NPN_CBE
- added Q2: BC847, Package_TO_SOT_SMD:SOT-23, symbol Transistor_BJT:BC847
Connections:
- net +12V: now also Q2.3 (C)
- net at R6.2, R7.1, R8.1: now also Q2.1 (B)
- net at D4.2 (A), R9.1: now also Q2.2 (E)
- net at C5.1, R11.1, U1.6 (-): no longer Q3.5 (B2), R15.2
- new net: Q3.5 (B2), R15.2
Changed lines of the file:
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@@
   (junction (at 149.86 189.23) (diameter 0) (color 0 0 0 0)
   )
+  (junction (at 161.29 171.45) (diameter 0) (color 0 0 0 0)
+  )
+  (junction (at 125.73 179.07) (diameter 0) (color 0 0 0 0)
+  )
+  (junction (at 218.44 90.17) (diameter 0) (color 0 0 0 0)
+  )
+  (junction (at 186.69 71.12) (diameter 0) (color 0 0 0 0)
+  )
+  (junction (at 231.14 62.23) (diameter 0) (color 0 0 0 0)
+  )
+  (junction (at 49.53 114.3) (diameter 0) (color 0 0 0 0)
+  )
+  (junction (at 199.39 114.3) (diameter 0) (color 0 0 0 0)
+  )
+  (junction (at 180.34 34.29) (diameter 0) (color 0 0 0 0)
+  )
+  (junction (at 267.97 146.05) (diameter 0) (color 0 0 0 0)
+  )
+  (junction (at 199.39 101.6) (diameter 0) (color 0 0 0 0)
+  )
+  (junction (at 125.73 72.39) (diameter 0) (color 0 0 0 0)
+  )
+  (junction (at 120.65 63.5) (diameter 0) (color 0 0 0 0)
+  )
+  (junction (at 215.9 54.61) (diameter 0) (color 0 0 0 0)
+  )
+  (junction (at 233.68 111.76) (diameter 0) (color 0 0 0 0)
+  )
   (junction (at 92.71 111.76) (diameter 0) (color 0 0 0 0)
   )
-  (junction (at 161.29 171.45) (diameter 0) (color 0 0 0 0)
-  )
-  (junction (at 125.73 179.07) (diameter 0) (color 0 0 0 0)
-  )
-  (junction (at 218.44 90.17) (diameter 0) (color 0 0 0 0)
-  )
-  (junction (at 186.69 71.12) (diameter 0) (color 0 0 0 0)
-  )
-  (junction (at 231.14 62.23) (diameter 0) (color 0 0 0 0)
-  )
-  (junction (at 49.53 114.3) (diameter 0) (color 0 0 0 0)
-  )
-  (junction (at 199.39 114.3) (diameter 0) (color 0 0 0 0)
-  )
-  (junction (at 180.34 34.29) (diameter 0) (color 0 0 0 0)
-  )
-  (junction (at 267.97 146.05) (diameter 0) (color 0 0 0 0)
-  )
-  (junction (at 199.39 101.6) (diameter 0) (color 0 0 0 0)
-  )
-  (junction (at 125.73 72.39) (diameter 0) (color 0 0 0 0)
-  )
-  (junction (at 120.65 63.5) (diameter 0) (color 0 0 0 0)
-  )
-  (junction (at 215.9 54.61) (diameter 0) (color 0 0 0 0)
-  )
-  (junction (at 233.68 111.76) (diameter 0) (color 0 0 0 0)
-  )
   (junction (at 215.9 43.18) (diameter 0) (color 0 0 0 0)
   )
@@
   )
   (junction (at 125.73 63.5) (diameter 0) (color 0 0 0 0)
-  )
-  (junction (at 160.02 68.58) (diameter 0) (color 0 0 0 0)
   )
   (junction (at 203.2 114.3) (diameter 0) (color 0 0 0 0)
@@
     (stroke (width 0) (type default))
   )
-  (wire (pts (xy 160.02 55.88) (xy 160.02 68.58))
-    (stroke (width 0) (type default))
-  )
   (wire (pts (xy 148.59 156.21) (xy 158.75 156.21))
     (stroke (width 0) (type default))
@@
     (stroke (width 0) (type default))
   )
-  (wire (pts (xy 160.02 68.58) (xy 160.02 101.6))
+  (wire (pts (xy 160.02 55.88) (xy 160.02 101.6))
     (stroke (width 0) (type default))
   )
@@
     )
   )
+  (symbol (lib_id "Transistor_BJT:BC847") (at 97.79 111.76 0) (unit 1)
+    (in_bom yes) (on_board yes) (dnp no) (fields_autoplaced)
+    (property "Reference" "Q2" (at 102.87 110.49 0)
+      (effects (font (size 1.27 1.27)) (justify left))
+    )
+    (property "Value" "BC847" (at 102.87 113.03 0)
+      (effects (font (size 1.27 1.27)) (justify left))
+    )
+    (property "Footprint" "Package_TO_SOT_SMD:SOT-23" (at 102.87 113.665 0)
+      (effects (font (size 1.27 1.27) italic) (justify left) hide)
+    )
+    (property "Datasheet" "http://www.infineon.com/dgdl/Infineon-BC847SERIES_BC848SERIES_BC849SERIES_BC850SERIES-DS-v01_01-en.pdf?fileId=db3a304314dca389011541d4630a1657" (at 97.79 111.76 0)
+      (effects (font (size 1.27 1.27)) (justify left) hide)
+    )
+    (property "Vendor" "Mouser" (at 97.79 111.76 0)
+      (effects (font (size 1.27 1.27)) hide)
+    )
+    (property "PartNum" "621-BC847C-13-F" (at 97.79 111.76 0)
+      (effects (font (size 1.27 1.27)) hide)
+    )
+    (pin "2")
+    (pin "1")
+    (pin "3")
+    (instances
+      (project "kick-drum"
+        (path "/54607e40-577c-4def-b17c-96859aef0795"
+          (reference "Q2") (unit 1)
+        )
+      )
+    )
+  )
   (symbol (lib_id "Mechanical:MountingHole_Pad") (at 59.69 185.42 0) (unit 1)
     (in_bom no) (on_board yes) (dnp no)
@@
         )
       )
-    )
-  )
-  (symbol (lib_id "Device:Q_NPN_CBE") (at 97.79 111.76 0) (unit 1)
-    (in_bom yes) (on_board yes) (dnp no)
-    (property "Reference" "Q2" (at 102.87 110.49 0)
-      (effects (font (size 1.27 1.27)) (justify left))
-    )
-    (property "Value" "BC547C" (at 102.87 113.03 0)
-      (effects (font (size 1.27 1.27)) (justify left))
-    )
-    (property "Footprint" "Package_TO_SOT_SMD:SOT-23-3" (at 102.87 109.22 0)
-      (effects (font (size 1.27 1.27)) hide)
-    )
-    (property "Datasheet" "~" (at 97.79 111.76 0)
-      (effects (font (size 1.27 1.27)) hide)
-    )
-    (property "Vendor" "Mouser" (at 97.79 111.76 0)
-      (effects (font (size 1.27 1.27)) hide)
-    )
-    (property "PartNum" "621-BC847C-13-F" (at 97.79 111.76 0)
-      (effects (font (size 1.27 1.27)) hide)
-    )
-    (pin "1")
-    (pin "3")
-    (pin "2")
-    (instances
-      (project "kick-drum"
-        (path "/54607e40-577c-4def-b17c-96859aef0795"
-          (reference "Q2") (unit 1)
-        )
-      )
